File: LiPo Power Packs/QT Backpack.brd (EAGLE design)
At the start: 30 x 17.7 mm, 14 parts, among them U1 TLV75533PDBVRDBV5_TEX-L, U2 MCP73831T-2ACI/OT

Commit message: Add files via upload
making sure current files are up to date.
Parts:
- R3: value 2K2 -> 2K
Changed lines of the file:
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@@
 <drawing>
 <settings>
-<setting alwaysvectorfont="yes"/>
+<setting alwaysvectorfont="no"/>
 <setting verticaltext="up"/>
 </settings>
@@
 <attribute name="VALUE" x="23.2896" y="14.4008" size="0.6096" layer="27" font="vector" ratio="20"/>
 </element>
-<element name="R3" library="rcl" library_urn="urn:adsk.eagle:library:334" package="R0603" package3d_urn="urn:adsk.eagle:package:23555/3" value="2K2" x="12.9794" y="7.62" smashed="yes" rot="R180">
+<element name="R3" library="rcl" library_urn="urn:adsk.eagle:library:334" package="R0603" package3d_urn="urn:adsk.eagle:package:23555/3" value="2K" x="12.9794" y="7.62" smashed="yes" rot="R180">
 <attribute name="NAME" x="11.3538" y="8.2804" size="1.27" layer="25" rot="R180"/>
 <attribute name="POPULARITY" value="77" x="-16.2306" y="25.4" size="1.778" layer="27" rot="R180" display="off"/>

Commit message: adding latest and JLCPCB CAM for 10pc panel
Parts:
- added U$1: MBR0520LT1G, MBR0520LT1G:SOD3716X117(SOD-123)
- moved CGD 12.2 mm to (18.4, 14.0), turned to 90 degrees
- moved CRG 11.8 mm to (18.5, 12.6), turned to 270 degrees
- moved J3 8.87 mm to (19.6, 6.68), turned to 270 degrees
- moved C3 5.19 mm to (12.7, 12.9)
- moved U2 4.94 mm to (12.5, 10.1)
- moved R2 4.50 mm to (8.71, 6.71)
- moved R1 4.42 mm to (8.68, 10.8)
- moved R3 4.42 mm to (8.71, 8.76)
- moved C4 4.42 mm to (8.68, 12.9)
- moved C2 2.98 mm to (4.75, 7.25)
- moved C1 2.54 mm to (4.86, 12.9)
- moved U1 2.32 mm to (4.88, 10.1)
Connections:
- new net +5V: C4.1, R1.2, U$1.2, U2.4
- net VUSB: now also U$1.1; no longer C4.1, R1.2, U2.4
Routing:
- net +5V: track 0.00 -> 16.5 mm, vias 0 -> 2
- net VUSB: track 18.3 -> 3.57 mm, vias 1 -> 0
- net VBAT: track 39.7 -> 25.6 mm, vias 2 -> 0
- net GND: track 0.00 -> 4.30 mm, vias 0 -> 34
- net N$18: track 11.3 -> 8.29 mm, vias 2 -> 0
- net N$24: track 9.53 -> 11.5 mm, vias 0 -> 2
- net N$25: track 14.7 -> 15.8 mm, vias 0 -> 2
- added copper zone on layer 16, net GND
Other:
- board size 30 x 17.7 mm -> 23.1 x 17.8 mm
- board text added: "LiPo Powerpack Rev B LiPo Charging/ Power For Qt Py Oak Dev Tech"
- board text removed: "BackPack Sapling LiPo Charging/Power For Qt Py Oak Dev Tech"
