File: LiPo Power Packs/QT Backpack.sch (EAGLE design)
At the start: 14 parts, among them U1 TLV75533PDBVRDBV5_TEX-L, U2 MCP73831T-2ACI/OT

Commit message: Add files via upload
making sure current files are up to date.
Parts:
- R3: value 2K2 -> 2K
Changed lines of the file:
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@@
 <parts>
 <part name="U2" library="MCP73831-2ACI" deviceset="MCP73831T-2ACI/OT" device=""/>
-<part name="R3" library="rcl" library_urn="urn:adsk.eagle:library:334" deviceset="R-US_" device="R0603" package3d_urn="urn:adsk.eagle:package:23555/3" value="2K2"/>
+<part name="R3" library="rcl" library_urn="urn:adsk.eagle:library:334" deviceset="R-US_" device="R0603" package3d_urn="urn:adsk.eagle:package:23555/3" value="2K"/>
 <part name="R1" library="rcl" library_urn="urn:adsk.eagle:library:334" deviceset="R-US_" device="R0603" package3d_urn="urn:adsk.eagle:package:23555/3" value="470"/>
 <part name="CRG" library="led" library_urn="urn:adsk.eagle:library:259" deviceset="LED" device="CHIP-LED0603" package3d_urn="urn:adsk.eagle:package:15819/3"/>

Commit message: adding latest and JLCPCB CAM for 10pc panel
Parts:
- added J4, J5: (no value), SparkFun-Connectors:CONN_07NO_SILK
- added SW: (no value), SparkFun-Connectors:CONN_02
- added U$1: MBR0520LT1G, MBR0520LT1G:MBR0520LT1G
- J1, J2: device SparkFun-Connectors:CONN_07NO_SILK -> SparkFun-Connectors:CONN_07LONGPADS
Connections:
- new net +5V: C4.1, R1.2, U$1.A, U2.VDD
- new net N$1: J2.7, J5.7
- new net N$3: J2.6, J5.6
- new net N$4: J2.5, J5.5
- new net N$5: J2.4, J5.4
- new net N$6: J2.3, J5.3
- new net N$7: J2.2, J5.2
- new net N$8: J2.1, J5.1
- net 3V: now also J4.5
- net GND: now also J4.6
- net VBAT: now also SW.1, SW.2
- net VUSB: now also J4.7, U$1.C; no longer C4.1, R1.2, U2.VDD
Other:
- note added: "Current as of Dec 8th, 2020"
- note added: "LiPo Power Pack"
- note added: "LiPo Power Pack designed to be pin compatible for use with the Adafruit Qt Py & Seeed Studio XIAO"
- note added: "MIT License"
- note added: "Oak Development Technologies"
- note added: "Oak Development Technologies LiPo Power Pack"
- moved on the sheet: J2
